Commit message: simulation works

File: model/urdf/plane_with_restitution.urdf (robot description, URDF)
Before this commit: robot plane, 1 links, 0 joints
Links:
- link planeLink: geometry collision box size=30 30 10; visual mesh filename=meshes/plane.obj scale=1 1 1

File: model/urdf/solo.urdf (robot description, URDF)
Before this commit: robot solo, 13 links, 12 joints
Links:
- link FL_FOOT: geometry collision mesh filename=meshes/stl/with_foot/solo_foot.stl; visual mesh filename=meshes/stl/with_foot/solo_foot.stl
- link FL_LOWER_LEG: geometry collision mesh filename=meshes/stl/with_foot/solo_lower_leg_left_side.stl; visual mesh filename=meshes/stl/with_foot/solo_lower_leg_left_side.stl
- link FL_UPPER_LEG: geometry collision mesh filename=meshes/stl/with_foot/solo_upper_leg_left_side.stl; visual mesh filename=meshes/stl/with_foot/solo_upper_leg_left_side.stl
- link FR_FOOT: geometry collision mesh filename=meshes/stl/with_foot/solo_foot.stl; visual mesh filename=meshes/stl/with_foot/solo_foot.stl
- link FR_LOWER_LEG: geometry collision mesh filename=meshes/stl/with_foot/solo_lower_leg_right_side.stl; visual mesh filename=meshes/stl/with_foot/solo_lower_leg_right_side.stl
- link FR_UPPER_LEG: geometry collision mesh filename=meshes/stl/with_foot/solo_upper_leg_right_side.stl; visual mesh filename=meshes/stl/with_foot/solo_upper_leg_right_side.stl
- link HL_FOOT: geometry collision mesh filename=meshes/stl/with_foot/solo_foot.stl; visual mesh filename=meshes/stl/with_foot/solo_foot.stl
- link HL_LOWER_LEG: geometry collision mesh filename=meshes/stl/with_foot/solo_lower_leg_left_side.stl; visual mesh filename=meshes/stl/with_foot/solo_lower_leg_left_side.stl
- link HL_UPPER_LEG: geometry collision mesh filename=meshes/stl/with_foot/solo_upper_leg_left_side.stl; visual mesh filename=meshes/stl/with_foot/solo_upper_leg_left_side.stl
- link HR_FOOT: geometry collision mesh filename=meshes/stl/with_foot/solo_foot.stl; visual mesh filename=meshes/stl/with_foot/solo_foot.stl
- link HR_LOWER_LEG: geometry collision mesh filename=meshes/stl/with_foot/solo_lower_leg_right_side.stl; visual mesh filename=meshes/stl/with_foot/solo_lower_leg_right_side.stl
- link HR_UPPER_LEG: geometry collision mesh filename=meshes/stl/with_foot/solo_upper_leg_right_side.stl; visual mesh filename=meshes/stl/with_foot/solo_upper_leg_right_side.stl
- link base_link: geometry collision mesh filename=meshes/stl/with_foot/solo_body.stl; visual mesh filename=meshes/stl/with_foot/solo_body.stl
